File: schematics/temp_arduino/temp_arduino.kicad_sch (KiCad schematic)
At the start: 0 parts

Commit message: update schematics
Parts:
- added A1: Arduino_UNO_R4(w/ wifi), Module:Arduino_UNO_R3, symbol MCU_Module:Arduino_UNO_R3
- added U1: ~, symbol shm_symbols:MCP9600_i2c_thermocouple_board
- added U2: ~, symbol shm_symbols:20x4_display
Connections:
- new net: A1.13 (SDA/A4), U1. (-), U2. (SCL)
- new net: A1.14 (SCL/A5), U1. (-), U2. (SCL)
- new net: A1.5 (+5V), U1. (-), U2. (SCL)
- new net: A1.7 (GND), U1. (-), U2. (SCL)

Commit message: update schematics
Parts:
- added TC1: Thermocouple, symbol Device:Thermocouple
- U1: value ~ -> MCP9600 i2c thermocouple board
- U2: value ~ -> 20x4 Display
Connections:
- net at U1. (-): now also TC1.2 (-)
- new net: A1.13 (SDA/A4), U1. (-), U2. (GND)
- new net: A1.14 (SCL/A5), U1. (-), U2. (GND)
- new net: A1.5 (+5V), U1. (-), U2. (GND)
- new net: TC1.1 (+), U1. (-)
Other:
- moved on the sheet: A1, U1, U2
