File: schematics/pi_control_of_shut_off/pi_control_of_shut_off/pi_control_of_shut_off.kicad_sch (KiCad schematic)
At the start: 0 parts

Commit message: update schematics
Parts:
- added J1: Raspberry_Pi_4, symbol Connector:Raspberry_Pi_4
- added R1: 10M, symbol Device:R
- added R2, R4: 330, symbol Device:R
- added R3: 100, symbol Device:R
- added R5: 47, symbol Device:R
- added SW1: AUTO ON SWITCH, symbol Switch:SW_Push
- added SW2: PUMP OFF SWITCH, symbol Switch:SW_Push
- added SW3: MANUAL ON SWITCH, symbol Switch:SW_Push
- added U1, U2: TLP3542, Package_DIP:DIP-5-6_W7.62mm, symbol Relay_SolidState:TLP3542
- added U3: Motor contactor, symbol shm_symbols:motor_contactor
Connections:
- new net: J1.1 (3V3), J1.17 (3V3)
- new net: J1.14 (GND), J1.20 (GND), J1.25 (GND), J1.30 (GND), J1.34 (GND), J1.39 (GND), J1.6 (GND), J1.9 (GND), R1.1, R5.2, SW2.1, U1.2, U1.4, U3. (MOTOR3)
- new net: J1.2 (5V), J1.4 (5V), SW1.1, SW3.1, U2.6
- new net: J1.29 (GPCLK1/GPIO05), R3.1
- new net: R3.2, U1.1
- new net: R5.1, U2.2
- new net: R1.2, R2.1, R4.1, SW2.2, U1.6, U2.1, U2.4, U3. (MOTOR3)
- new net: R2.2, SW1.2
- new net: R4.2, SW3.2
