File: schematics/tank_pi/tank_pi.kicad_sch (KiCad schematic)
At the start: 0 parts

Commit message: update schematics
Parts:
- added J1: Raspberry_Pi_4, symbol Connector:Raspberry_Pi_4
- added U1: Roadside sensor, symbol shm_symbols:Ultrasonic_distance_sensor
- added U2: Brookside sensor, symbol shm_symbols:Ultrasonic_distance_sensor
- added U3: Adafruit i2c 16x2 RGB LCD Pi Plate, symbol shm_symbols:16x2_RGB_LCD_Pi_Plate
Connections:
- new net: J1.1 (3V3), J1.17 (3V3)
- new net: J1.10 (GPIO15/UART_RXD), U2. (M2)
- new net: J1.14 (GND), J1.20 (GND), J1.25 (GND), J1.30 (GND), J1.34 (GND), J1.39 (GND), J1.6 (GND), J1.9 (GND), U1. (M2), U2. (M2)
- new net: J1.2 (5V), J1.4 (5V), U1. (M2), U2. (M2)
- new net: J1.32 (GPIO12/PWM0), U1. (M2)
- new net: J1.33 (GPIO13/PWM1), U1. (M2)
- new net: J1.8 (GPIO14/UART_TXD), U2. (M2)

Commit message: update schematics
Other:
- moved on the sheet: U1, U2, U3
